Commit message: Commit message

File: install/robotic_arm/share/robotic_arm/urdf/robotic_arm.urdf (robot description, URDF)
Before this commit: robot robotic_arm, 7 links, 6 joints
Links:
- added link camera_link, mass 0.01; collision box size=0.05 0.05 0.05; visual box size=0.05 0.05 0.05
Joints:
- added joint camera_joint: type fixed, parent link_3, child camera_link, origin xyz=0 0 0.4 rpy=0 0 0

Commit message: controller changed

File: install/robotic_arm/share/robotic_arm/urdf/robotic_arm.urdf (robot description, URDF)
Before this commit: robot robotic_arm, 8 links, 7 joints
Links:
- link camera_link: mass 0.01 -> 1e-5; geometry collision box size=${camera_link} ${camera_link} ${camera_link}; visual box size=${camera_link} ${camera_link} ${camera_link}
Joints:
- joint camera_joint: axis (none) -> 0 1 0; origin xyz=0 0 0.4 rpy=0 0 0 -> xyz=0 0 0 rpy=0 0 0
